File: Kicad/RLab Keyboard/RLab Keyboard.kicad_pcb (KiCad board)
At the start: 2 copper layers, 100 x 100 mm, 81 parts, among them J1 Conn_01x01_Pin, J10 Conn_01x01_Pin, J11 Conn_01x01_Pin, J12 Conn_01x01_Pin, J13 Conn_01x07, J14 Conn_01x09, J15 Conn_01x09, J16 Conn_01x09, J17 AudioJack3_Switch, J18 Conn_01x06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

Commit message: Files updated for JLCPCB Assembly
Added DNP  for through hole components. can be viewed as option in 3D viewer.
Production files in JLCPCB folder
Parts:
- D1, D2, D3: value D -> 1N5819WS
